File: Hardware/SPI2TTL/FPGA.kicad_sch (KiCad schematic)
At the start: 98 parts, among them J1 Conn_01x06, J7 Conn_02x07_Odd_Even, J8 Conn_01x40, SW1 SW_Push, SW2 SW_Push, SW3 SW_Push, SW4 SW_DIP_x03, U1 XC7S15-2CSGA225I, U2 IS25LP032D, X1 SG-5032CBN

Commit message: Updated SCH & PCB with corrected CLK traces, BOM and gerbers
Parts:
- C18: value 15pF -> DNP
- R36, R37, R38, R39: value 1K -> 3.3K
- R40, R41: value 4.7K -> 1K
- R5: value 200R -> 3.3K
- R52, R53: value 4.7K -> DNP
Connections:
- no-connect marks 71 -> 77
Changed lines of the file:
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@@
 	)
 	(no_connect
+		(at 132.08 137.16)
+	)
+	(no_connect
 		(at 506.73 214.63)
 	)
@@
 	)
 	(no_connect
+		(at 318.77 114.3)
+	)
+	(no_connect
 		(at 132.08 73.66)
 	)
@@
 	)
 	(no_connect
+		(at 132.08 134.62)
+	)
+	(no_connect
+		(at 318.77 104.14)
+	)
+	(no_connect
 		(at 481.33 240.03)
 	)
 	(no_connect
+		(at 318.77 116.84)
+	)
+	(no_connect
 		(at 318.77 40.64)
 	)
@@
 	)
 	(no_connect
+		(at 132.08 142.24)
+	)
+	(no_connect
 		(at 481.33 212.09)
 	)
@@
 			)
 		)
-		(property "Value" "1K"
+		(property "Value" "3.3K"
 			(at 59.69 229.87 90)
 			(effects
@@
 			)
 		)
-		(property "Value" "4.7K"
+		(property "Value" "1K"
 			(at 125.095 204.47 0)
 			(effects
@@
 			)
 		)
-		(property "Value" "1K"
+		(property "Value" "3.3K"
 			(at 59.69 204.47 90)
 			(effects
@@
 			)
 		)
-		(property "Value" "1K"
+		(property "Value" "3.3K"
 			(at 59.69 217.17 90)
 			(effects
@@
 			)
 		)
-		(property "Value" "4.7K"
+		(property "Value" "DNP"
 			(at 152.4 380.9999 0)
 			(effects
@@
 			)
 		)
-		(property "Value" "4.7K"
+		(property "Value" "1K"
 			(at 125.095 237.49 0)
 			(effects
@@
 			)
 		)
-		(property "Value" "200R"
+		(property "Value" "3.3K"
 			(at 110.49 318.7699 0)
 			(effects
@@
 			)
 		)
-		(property "Value" "4.7K"
+		(property "Value" "DNP"
 			(at 95.25 59.6899 0)
 			(effects
@@
 			)
 		)
-		(property "Value" "1K"
+		(property "Value" "3.3K"
 			(at 59.69 242.57 90)
 			(effects
@@
 			)
 		)
-		(property "Value" "15pF"
+		(property "Value" "DNP"
 			(at 187.96 381.0062 0)
 			(effects
