File: Hardware/SPI2TTL/Power.kicad_sch (KiCad schematic)
At the start: 24 parts, among them U5 TLV76701DRVR, U6 TLV76701DRVR, U7 TLV76701DRVR, U8 TLV61046ADB

Commit message: Updated SCH & PCB with corrected CLK traces, BOM and gerbers
Parts:
- C47, C50, C53: now fitted
Changed lines of the file:
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@@
 		(in_bom yes)
 		(on_board yes)
-		(dnp yes)
+		(dnp no)
 		(fields_autoplaced yes)
 		(property "Reference" "C53"
@@
 		(in_bom yes)
 		(on_board yes)
-		(dnp yes)
+		(dnp no)
 		(fields_autoplaced yes)
 		(property "Reference" "C50"
@@
 		(in_bom yes)
 		(on_board yes)
-		(dnp yes)
+		(dnp no)
 		(fields_autoplaced yes)
 		(property "Reference" "C47"
